File: schematic/led-bottle-lighting.kicad_pcb (KiCad board)
At the start: 2 copper layers, 13 parts, among them J1 Barrel_Jack, J2 Conn_01x03_Female, J3 Conn_01x02, Q1 Q_NMOS_DSG, U1 LM7805_TO220, U2 WeMos_D1_mini

Commit message: imp: update schematic
Parts:
- moved U2 8.03 mm to (137.2, 149.9)
- moved J2 6.35 mm to (142.2, 121.9)
- moved R3 5.68 mm to (106.7, 106.7), turned to 180 degrees
- moved Q1 5.68 mm to (99.1, 139.7)
- moved R1 3.81 mm to (109.2, 148.6)
- moved R2 2.54 mm to (109.2, 144.8)
- turned D1 to 0 degrees
Routing:
- net +5V: track 17.3 -> 66.3 mm, vias 0 -> 3
- net Touch_S: track 0.00 -> 45.7 mm
- net +3V3: track 0.00 -> 22.9 mm
- net GATE: track 0.00 -> 21.6 mm
- net +12V: track 33.6 -> 50.1 mm, vias 0 -> 2
- net Net-(Q1-Pad3): track 0.00 -> 14.0 mm
- net LED_K: track 0.00 -> 12.7 mm
- net Net-(D1-Pad2): track 5.08 -> 2.54 mm
- net GND: track 113.2 -> 111.9 mm
